File: PCB/Base PCB/PCB.kicad_sch (KiCad schematic)
At the start: 14 parts, among them J1 Conn_01x19_Socket, J10 Conn_01x01_Socket, J2 Conn_01x19_Socket, J3 Conn_01x03_Socket, J4 Conn_01x01_Socket, J5 Conn_01x01_Socket, J6 Conn_01x01_Socket, J7 Conn_01x01_Socket, J8 Conn_01x01_Socket, J9 Conn_01x01_Socket

Commit message: Finished the rough draft for the enclosure. I used the 3d models from KiCad to get the PCB dimensions.
Parts:
- removed J10, J4, J9: Conn_01x01_Socket, Connector_PinHeader_2.54mm:PinHeader_1x01_P2.54mm_Vertical, symbol Connector:Conn_01x01_Socket
- added J4: Conn_01x09_Socket, Connector_PinHeader_2.54mm:PinHeader_1x09_P2.54mm_Vertical, symbol Connector:Conn_01x09_Socket
Connections:
- net 13: now also J3.1 (Pin_1)
- net 14: now also J4.7 (Pin_7)
- net 27: now also J4.6 (Pin_6)
- net 32: now also J4.4 (Pin_4); no longer J7.1 (Pin_1)
- net 33: now also J4.5 (Pin_5); no longer J8.1 (Pin_1)
- net 34: now also J4.2 (Pin_2); no longer J5.1 (Pin_1)
- net 35: now also J4.3 (Pin_3); no longer J6.1 (Pin_1)
- net 36: no longer J3.1 (Pin_1)
- net 39: now also J4.1 (Pin_1)
- net 5V: now also J3.3 (Pin_3), J6.1 (Pin_1), J4.9 (Pin_9); no longer J3.2 (Pin_2)
- net GND: now also J3.2 (Pin_2), J5.1 (Pin_1), J4.8 (Pin_8); no longer J3.3 (Pin_3)
- new net B_5V: J8.1 (Pin_1)
- new net B_GND: J7.1 (Pin_1)
Other:
- note added: "Button 1 sockets"
- note added: "Port sockets"
- note added: "Power sockets"
